File: medidor de capacitancia.kicad_sch (KiCad schematic)
At the start: 6 parts, among them Q1 BC327, U1 RP2040

Commit message: Add files via upload
Parts:
- removed Q1: BC327, Package_TO_SOT_THT:TO-92_Inline, symbol Transistor_BJT:BC327
Connections:
- net at R1.1: now also C1.1, R2.1, R3.1
- net at R1.2: now also U1.23 (DVDD), U1.50 (DVDD)
- net at R3.2: now also U1.48 (USB_VDD)
- net at U1.1 (IOVDD), U1.10 (IOVDD), U1.22 (IOVDD)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: now also R2.2
Other:
- moved on the sheet: R1, R2, R3
Changed lines of the file:
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@@
 	(generator_version "8.0")
 	(paper "A4")
-	(wire
-		(pts
-			(xy 97.79 58.42) (xy 113.03 58.42)
+	(junction
+		(at 92.71 27.94)
+		(diameter 0)
+		(color 0 0 0 0)
+	)
+	(junction
+		(at 93.98 27.94)
+		(diameter 0)
+		(color 0 0 0 0)
+	)
+	(wire
+		(pts
+			(xy 71.12 38.1) (xy 71.12 31.75)
+		)
+		(stroke
+			(width 0)
+			(type default)
+		)
+	)
+	(wire
+		(pts
+			(xy 63.5 24.13) (xy 86.36 24.13)
+		)
+		(stroke
+			(width 0)
+			(type default)
+		)
+	)
+	(wire
+		(pts
+			(xy 63.5 38.1) (xy 63.5 24.13)
 		)
 		(stroke
@@
 	(wire
 		(pts
-			(xy 91.44 63.5) (xy 107.95 63.5)
+			(xy 68.58 38.1) (xy 68.58 27.94)
+		)
+		(stroke
+			(width 0)
+			(type default)
+		)
+	)
+	(wire
+		(pts
+			(xy 92.71 27.94) (xy 92.71 31.75)
+		)
+		(stroke
+			(width 0)
+			(type default)
+		)
+	)
+	(wire
+		(pts
+			(xy 68.58 27.94) (xy 85.09 27.94)
+		)
+		(stroke
+			(width 0)
+			(type default)
+		)
+	)
+	(wire
+		(pts
+			(xy 93.98 27.94) (xy 123.19 27.94)
 		)
 		(stroke
@@
 	(wire
 		(pts
-			(xy 91.44 53.34) (xy 97.79 53.34)
-		)
-		(stroke
-			(width 0)
-			(type default)
-		)
-	)
-	(wire
-		(pts
-			(xy 107.95 66.04) (xy 118.11 66.04)
+			(xy 71.12 31.75) (xy 85.09 31.75)
 		)
 		(stroke
@@
 	(wire
 		(pts
-			(xy 107.95 63.5) (xy 107.95 66.04)
-		)
-		(stroke
-			(width 0)
-			(type default)
-		)
-	)
-	(wire
-		(pts
-			(xy 97.79 53.34) (xy 97.79 58.42)
+			(xy 93.98 24.13) (xy 93.98 27.94)
+		)
+		(stroke
+			(width 0)
+			(type default)
+		)
+	)
+	(wire
+		(pts
+			(xy 92.71 27.94) (xy 93.98 27.94)
+		)
+		(stroke
+			(width 0)
+			(type default)
+		)
+	)
+	(wire
+		(pts
+			(xy 123.19 58.42) (xy 123.19 27.94)
 		)
 		(stroke
@@
 	(symbol
 		(lib_id "Device:R")
-		(at 129.54 46.99 0)
+		(at 90.17 24.13 0)
 		(unit 1)
 		(exclude_from_sim no)
@@
 		(fields_autoplaced yes)
 		(property "Reference" "R1"
-			(at 129.54 40.64 0)
+			(at 90.17 17.78 0)
 			(effects
 				(font
@@
 		)
 		(property "Value" "R"
-			(at 129.54 43.18 0)
+			(at 90.17 20.32 0)
 			(effects
 				(font
@@
 		)
 		(property "Footprint" ""
-			(at 129.54 45.212 0)
+			(at 90.17 22.352 0)
 			(effects
 				(font
@@
 		)
 		(property "Datasheet" "~"
-			(at 129.54 46.99 90)
+			(at 90.17 24.13 90)
 			(effects
 				(font
@@
 		)
 		(property "Description" "Resistor"
-			(at 129.54 46.99 0)
+			(at 90.17 24.13 0)
 			(effects
 				(font
@@
 	(symbol
 		(lib_id "Device:R")
-		(at 142.24 46.99 0)
+		(at 88.9 31.75 0)
 		(unit 1)
 		(exclude_from_sim no)
@@
 		(fields_autoplaced yes)
 		(property "Reference" "R3"
-			(at 142.24 40.64 0)
+			(at 88.9 25.4 0)
 			(effects
 				(font
@@
 		)
 		(property "Value" "R"
-			(at 142.24 43.18 0)
+			(at 88.9 27.94 0)
 			(effects
 				(font
@@
 		)
 		(property "Footprint" ""
-			(at 142.24 45.212 0)
+			(at 88.9 29.972 0)
 			(effects
 				(font
@@
 		)
 		(property "Datasheet" "~"
-			(at 142.24 46.99 90)
+			(at 88.9 31.75 90)
 			(effects
 				(font
@@
 		)
 		(property "Description" "Resistor"
-			(at 142.24 46.99 0)
+			(at 88.9 31.75 0)
 			(effects
 				(font
@@
 				(path "/5ec8c912-b8bb-4493-a652-567182c58a72"
 					(reference "R3")
-					(unit 1)
-				)
-			)
-		)
-	)
-	(symbol
-		(lib_id "Transistor_BJT:BC327")
-		(at 118.11 60.96 90)
-		(unit 1)
-		(exclude_from_sim no)
-		(in_bom yes)
-		(on_board yes)
-		(dnp no)
-		(property "Reference" "Q1"
-			(at 116.8399 55.88 0)
-			(effects
-				(font
-					(size 1.27 1.27)
-				)
-				(justify left)
-			)
-		)
-		(property "Value" "BC327"
-			(at 119.3799 55.88 0)
-			(effects
-				(font
-					(size 1.27 1.27)
-				)
-				(justify left)
-			)
-		)
-		(property "Footprint" "Package_TO_SOT_THT:TO-92_Inline"
-			(at 120.015 55.88 0)
-			(effects
-				(font
-					(size 1.27 1.27)
-					(italic yes)
-				)
-				(justify left)
-				(hide yes)
-			)
-		)
-		(property "Datasheet" "http://www.onsemi.com/pub_link/Collateral/BC327-D.PDF"
-			(at 118.11 60.96 0)
-			(effects
-				(font
-					(size 1.27 1.27)
-				)
-				(justify left)
-				(hide yes)
-			)
-		)
-		(property "Description" "0.8A Ic, 45V Vce, PNP Transistor, TO-92"
-			(at 118.11 60.96 0)
-			(effects
-				(font
-					(size 1.27 1.27)
-				)
-				(hide yes)
-			)
-		)
-		(pin "3"
-		)
-		(pin "2"
-		)
-		(pin "1"
-		)
-		(instances
-			(project ""
-				(path "/5ec8c912-b8bb-4493-a652-567182c58a72"
-					(reference "Q1")
 					(unit 1)
 				)
@@
 	(symbol
 		(lib_id "Device:R")
-		(at 119.38 44.45 0)
+		(at 88.9 27.94 0)
 		(unit 1)
 		(exclude_from_sim no)
@@
 		(fields_autoplaced yes)
 		(property "Reference" "R2"
-			(at 119.38 38.1 0)
+			(at 88.9 21.59 0)
 			(effects
 				(font
@@
 		)
 		(property "Value" "R"
-			(at 119.38 40.64 0)
+			(at 88.9 24.13 0)
 			(effects
 				(font
@@
 		)
 		(property "Footprint" ""
-			(at 119.38 42.672 0)
+			(at 88.9 26.162 0)
 			(effects
 				(font
@@
 		)
 		(property "Datasheet" "~"
-			(at 119.38 44.45 90)
+			(at 88.9 27.94 90)
 			(effects
 				(font
@@
 		)
 		(property "Description" "Resistor"
-			(at 119.38 44.45 0)
-			(effects
-				(font
+			(at 88.9 27.94 0)
+			(effects
+				(font
